Commit message: 20220425

File: my_ur_description/urdf/ur3/ur3_robot.urdf.xacro (robot description, xacro)
@@ -90,5 +90,5 @@
     <parent link="tool0" />
     <child link="tcp_link" />
-    <origin xyz="0.0 0.0 0.0" rpy="0.0 ${-pi/2} 0.0"/>
+    <origin xyz="0.0 0.0 0.08" rpy="0.0 ${-pi/2} 0.0"/>
   </joint>
   <link name="beugel_base_position"/>
@@ -110,5 +110,8 @@
     <parent link="beugel_link" />
     <child link="beugel_camera_position" />
+    <!--
     <origin xyz="0.0 -0.0049 0.0507" rpy="3.14 ${pi/6+3.14} -${pi/2}"/>
+    -->
+    <origin xyz="0.0 -0.0049 0.0507" rpy="0.0 ${pi/6} -${pi/2}"/>
   </joint>
  <link name="camera_mouniting_holes"/>
@@ -122,4 +125,10 @@
     <origin xyz="0.0 0 0" rpy="0.0 0 0"/>
   </xacro:sensor_d435>
-  <xacro:vacuum_tool prefix="" connected_to="tool0"/>
+  <link name = "gripper_base_link"/>
+  <joint name="beugel_to_gripper" type ="fixed">
+      <parent link="tool0" />
+      <child link="gripper_base_link" />
+      <origin xyz="0.0 0.0 0.003" rpy="0.0 0.0 0.0"/>
+  </joint>
+  <xacro:vacuum_tool prefix="" connected_to="gripper_base_link"/>
 </robot>

Commit message: 202200505

File: my_ur_description/urdf/ur3/ur3_robot.urdf.xacro (robot description, xacro)
@@ -3,7 +3,7 @@
   <xacro:include filename="$(find ur_description)/urdf/inc/ur3_macro.xacro"/>
   <!-- bracket/beugel -->
-  <xacro:include filename="$(find urdf_support)/beugel/urdf/Beugel.urdf.xacro" />
+  <xacro:include filename="$(find pcl_urdf_support)/beugel/urdf/Beugel.urdf.xacro" />
   <xacro:beugel/>
-  <xacro:include filename="$(find urdf_support)/avans_vacuum_gripper/urdf/avans_vacuum_gripper.xacro" />
+  <xacro:include filename="$(find avans_vacuum_gripper_urdf_support)/avans_vacuum_gripper/urdf/avans_vacuum_gripper.xacro" />
   <!-- camera -->
   <xacro:include filename="$(find realsense2_description)/urdf/_d435.urdf.xacro" />
@@ -110,8 +110,8 @@
     <parent link="beugel_link" />
     <child link="beugel_camera_position" />
+    <origin xyz="0.0 -0.0049 0.0507" rpy="3.14 ${pi/6+3.14} -${pi/2}"/>
     <!--
-    <origin xyz="0.0 -0.0049 0.0507" rpy="3.14 ${pi/6+3.14} -${pi/2}"/>
-    -->
     <origin xyz="0.0 -0.0049 0.0507" rpy="0.0 ${pi/6} -${pi/2}"/>
+  -->
   </joint>
  <link name="camera_mouniting_holes"/>

Commit message: 20220509

File: my_ur_description/urdf/ur3/ur3_robot.urdf.xacro (robot description, xacro)
@@ -115,14 +115,17 @@
   -->
   </joint>
- <link name="camera_mouniting_holes"/>
- <joint name="camera_mouniting_holes_to_beugel_camera_position" type="fixed">
+ <link name="camera_mounting_holes"/>
+ <joint name="camera_mounting_holes_to_beugel_camera_position" type="fixed">
     <parent link="beugel_camera_position" />
-    <child link="camera_mouniting_holes" />
+    <child link="camera_mounting_holes" />
     <origin xyz="-0.006 0.0 -0.006" rpy="0.0 0.0 0"/> <!-- deze waardes zijn nog niet geheel juist, natrekken bij mechanische tekeningen camera-->
  </joint>
   <!-- camera_to robot -->
-  <xacro:sensor_d435 parent="camera_mouniting_holes" use_nominal_extrinsics="true">
-    <origin xyz="0.0 0 0" rpy="0.0 0 0"/>
+  <xacro:sensor_d435 parent="camera_mounting_holes" use_nominal_extrinsics="true">
+    <origin xyz="0.011 0.000 0.000" rpy="0.0 0 0"/>
   </xacro:sensor_d435>
+<!--
+0.011, 0.018, 0.013
+-->
   <link name = "gripper_base_link"/>
   <joint name="beugel_to_gripper" type ="fixed">
